Commit message: complete package change for robot for compatible configurement

File: install/unitree_go2_description/share/unitree_go2_description/urdf/unitree_go2_gazebo.xacro (robot description, xacro)
@@ -1 +1,224 @@
-/home/ming/ros2_ws/src/unitree_go2/unitree_go2_description/urdf/unitree_go2_gazebo.xacro
+<?xml version="1.0"?>
+<robot xmlns:xacro="http://ros.org/wiki/xacro">
+<xacro:macro name="unitree_go2_gazebo" params="robot_controllers">
+  <!-- Gazebo Sim plugins -->
+  <gazebo>
+    <plugin filename="gz-sim-pose-publisher-system" name="gz::sim::systems::PosePublisher">
+      <publish_link_pose>true</publish_link_pose>
+      <publish_sensor_pose>true</publish_sensor_pose>
+      <publish_collision_pose>false</publish_collision_pose>
+      <publish_visual_pose>false</publish_visual_pose>
+      <publish_nested_model_pose>false</publish_nested_model_pose>
+      <use_pose_vector_msg>true</use_pose_vector_msg>
+      <static_publisher>true</static_publisher>
+      <static_update_frequency>100</static_update_frequency>
+    </plugin>
+  </gazebo>
+        <!-- Robot-wide physics properties -->
+        <!-- <gazebo>
+            <plugin filename="gz-sim-physics-system" name="gz::sim::systems::Physics">
+                <engine>
+                    <filename>gz-physics-bullet-plugin</filename>
+                </engine>
+            </plugin>
+        </gazebo> -->
+  <!-- ROS2 Control plugin -->
+  <gazebo>
+    <plugin filename="gz_ros2_control-system" name="gz_ros2_control::GazeboSimROS2ControlPlugin">
+      <parameters>${robot_controllers}</parameters>
+      <robot_param_node>robot_state_publisher</robot_param_node>
+    </plugin>
+  </gazebo>
+        <!-- Odometry plugin - DISABLED (broken on this system)
+        <gazebo>
+            <plugin filename="gz-sim-odometry-publisher-system"
+                name="gz::sim::systems::OdometryPublisher">
+                <odom_frame>odom</odom_frame>
+                <robot_base_frame>base_link</robot_base_frame>
+                <odom_topic>/odom</odom_topic>
+                <odom_publish_frequency>50</odom_publish_frequency>
+            </plugin>
+        </gazebo>
+        -->
+        <!-- IMU plugin -->
+        <gazebo reference="imu_link">
+            <sensor name="imu_sensor" type="imu">
+                <always_on>true</always_on>
+                <update_rate>100</update_rate>
+                <visualize>true</visualize>
+                <topic>imu/data</topic>
+                <gz_frame_id>imu_link</gz_frame_id>
+                <imu>
+                    <angular_velocity>
+                        <x>
+                            <noise type="gaussian">
+                                <mean>0.0</mean>
+                                <stddev>2e-4</stddev>
+                            </noise>
+                        </x>
+                        <y>
+                            <noise type="gaussian">
+                                <mean>0.0</mean>
+                                <stddev>2e-4</stddev>
+                            </noise>
+                        </y>
+                        <z>
+                            <noise type="gaussian">
+                                <mean>0.0</mean>
+                                <stddev>2e-4</stddev>
+                            </noise>
+                        </z>
+                    </angular_velocity>
+                    <linear_acceleration>
+                        <x>
+                            <noise type="gaussian">
+                                <mean>0.0</mean>
+                                <stddev>1.7e-2</stddev>
+                            </noise>
+                        </x>
+                        <y>
+                            <noise type="gaussian">
+                                <mean>0.0</mean>
+                                <stddev>1.7e-2</stddev>
+                            </noise>
+                        </y>
+                        <z>
+                            <noise type="gaussian">
+                                <mean>0.0</mean>
+                                <stddev>1.7e-2</stddev>
+                            </noise>
+                        </z>
+                    </linear_acceleration>
+                </imu>
+                <plugin filename="gz-sim-imu-system" name="gz::sim::systems::Imu">
+                    <initial_orientation_as_reference>false</initial_orientation_as_reference>
+                </plugin>
+            </sensor>
+        </gazebo>
+        <!-- Camera Plugin-->
+        <gazebo reference="camera_link">
+            <sensor name="rgb_camera" type="camera">
+                <pose>0 0.0 0 0 0 0</pose>
+                <camera>
+                    <horizontal_fov>1.367</horizontal_fov>
+                    <image>
+                        <width>640</width>
+                        <height>480</height>
+                    </image>
+                    <clip>
+                        <near>0.05</near>
+                        <far>200</far>
+                    </clip>
+                </camera>
+                <gz_frame_id>camera_link</gz_frame_id>
+                <always_on>1</always_on>
+                <update_rate>10</update_rate>
+                <visualize>1</visualize>
+                <topic>rgb_image</topic>
+            </sensor>
+        </gazebo>
+        <!-- Main body -->
+        <gazebo reference="trunk">
+            <mu1>0.2</mu1>
+            <mu2>0.2</mu2>
+            <kp>10000.0</kp>
+            <kd>1.0</kd>
+        </gazebo>
+        <!-- FL leg -->
+        <gazebo reference="lf_hip_link">
+            <mu1>0.2</mu1>
+            <mu2>0.2</mu2>
+        </gazebo>
+        <gazebo reference="lf_upper_leg_link">
+            <mu1>0.2</mu1>
+            <mu2>0.2</mu2>
+            <self_collide>1</self_collide>
+            <kp>10000.0</kp>
+            <kd>1.0</kd>
+        </gazebo>
+        <gazebo reference="lf_lower_leg_link">
+            <mu1>0.2</mu1>
+            <mu2>0.2</mu2>
+            <self_collide>1</self_collide>
+        </gazebo>
+        <gazebo reference="lf_foot_link">
+            <mu1>0.6</mu1>
+            <mu2>0.6</mu2>
+            <self_collide>1</self_collide>
+            <kp>10000.0</kp>
+            <kd>1.0</kd>
+        </gazebo>
+        <!-- FR leg -->
+        <gazebo reference="rf_hip_link">
+            <mu1>0.2</mu1>
+            <mu2>0.2</mu2>
+        </gazebo>
+        <gazebo reference="rf_upper_leg_link">
+            <mu1>0.2</mu1>
+            <mu2>0.2</mu2>
+            <self_collide>1</self_collide>
+            <kp>10000.0</kp>
+            <kd>1.0</kd>
+        </gazebo>
+        <gazebo reference="rf_lower_leg_link">
+            <mu1>0.2</mu1>
+            <mu2>0.2</mu2>
+            <self_collide>1</self_collide>
+        </gazebo>
+        <gazebo reference="rf_foot_link">
+            <mu1>0.6</mu1>
+            <mu2>0.6</mu2>
+            <self_collide>1</self_collide>
+            <kp>10000.0</kp>
+            <kd>1.0</kd>
+        </gazebo>
+        <!-- RL leg -->
+        <gazebo reference="lh_hip_link">
+            <mu1>0.2</mu1>
+            <mu2>0.2</mu2>
+        </gazebo>
+        <gazebo reference="lh_upper_leg_link">
+            <mu1>0.2</mu1>
+            <mu2>0.2</mu2>
+            <self_collide>1</self_collide>
+            <kp>10000.0</kp>
+            <kd>1.0</kd>
+        </gazebo>
+        <gazebo reference="lh_lower_leg_link">
+            <mu1>0.2</mu1>
+            <mu2>0.2</mu2>
+            <self_collide>1</self_collide>
+        </gazebo>
+        <gazebo reference="lh_foot_link">
+            <mu1>0.6</mu1>
+            <mu2>0.6</mu2>
+            <self_collide>1</self_collide>
+            <kp>10000.0</kp>
+            <kd>1.0</kd>
+        </gazebo>
+  <!-- RR leg -->
+  <gazebo reference="rh_hip_link">
+    <mu1>0.2</mu1>
+    <mu2>0.2</mu2>
+  </gazebo>
+  <gazebo reference="rh_upper_leg_link">
+    <mu1>0.2</mu1>
+    <mu2>0.2</mu2>
+    <self_collide>1</self_collide>
+    <kp>10000.0</kp>
+    <kd>1.0</kd>
+  </gazebo>
+  <gazebo reference="rh_lower_leg_link">
+    <mu1>0.2</mu1>
+    <mu2>0.2</mu2>
+    <self_collide>1</self_collide>
+  </gazebo>
+  <gazebo reference="rh_foot_link">
+    <mu1>0.6</mu1>
+    <mu2>0.6</mu2>
+    <self_collide>1</self_collide>
+    <kp>10000.0</kp>
+    <kd>1.0</kd>
+  </gazebo>
+</xacro:macro>
+</robot>

File: install/unitree_go2_description/share/unitree_go2_description/urdf/unitree_go2_robot.xacro (robot description, xacro)
@@ -1 +1,149 @@
-/home/ming/ros2_ws/src/unitree_go2/unitree_go2_description/urdf/unitree_go2_robot.xacro
+<?xml version="1.0"?>
+<robot name="go2"
+    xmlns:xacro="http://www.ros.org/wiki/xacro">
+    <xacro:arg name="DEBUG" default="false"/>
+    <xacro:arg name="robot_controllers" default="$(find unitree_go2_sim)/config/ros_control/ros_control.yaml"/>
+    <xacro:include filename="$(find unitree_go2_description)/urdf/const.xacro" />
+    <xacro:include filename="$(find unitree_go2_description)/urdf/materials.xacro" />
+    <xacro:include filename="$(find unitree_go2_description)/urdf/leg.xacro" />
+    <!-- <xacro:include filename="$(find unitree_go2_description)/stairs.xacro"/> -->
+    <xacro:include filename="$(find unitree_go2_description)/urdf/unitree_go2_gazebo.xacro" />
+    <!-- <xacro:include filename="$(find unitree_go2_description)/launch/stairs.urdf.xacro"/> -->
+    <xacro:include filename="$(find unitree_go2_description)/urdf/velodyne.xacro"/>
+    <xacro:include filename="$(find unitree_go2_description)/urdf/lidar_4D_lidar.xacro"/>
+    <xacro:include filename="$(find unitree_go2_description)/urdf/realsense_d455.xacro"/>
+    <!-- <xacro:stairs stairs="15" xpos="0" ypos="0" zpos="0" /> -->
+    <xacro:unitree_go2_gazebo robot_controllers="$(arg robot_controllers)"/>
+    <!-- Rotor related joint and link is only for demonstrate location. -->
+    <!-- Actually, the rotor will rotate and the joint is not fixed. Reduction ratio should be
+    considered. -->
+    <!-- Debug mode will hung up the robot, use "true" or "false" to switch it. -->
+    <xacro:if value="$(arg DEBUG)">
+        <link name="world" />
+        <joint name="base_static_joint" type="fixed">
+            <origin rpy="0 0 0" xyz="0 0 0" />
+            <parent link="world" />
+            <child link="base_link" />
+        </joint>
+    </xacro:if>
+    <link name="base_link">
+        <visual>
+            <origin rpy="0 0 0" xyz="0 0 0" />
+            <geometry>
+                <box size="0.001 0.001 0.001" />
+            </geometry>
+        </visual>
+    </link>
+    <joint name="floating_base" type="fixed">
+        <origin rpy="0 0 0" xyz="0 0 0" />
+        <parent link="base_link" />
+        <child link="trunk" />
+    </joint>
+    <link name="trunk">
+        <visual>
+            <origin rpy="0 0 0" xyz="0 0 0" />
+            <geometry>
+                <mesh filename="file://$(find unitree_go2_description)/meshes/trunk.dae"
+                    scale="1 1 1" />
+            </geometry>
+        </visual>
+        <collision>
+            <origin rpy="0 0 0" xyz="0 0 0" />
+            <geometry>
+                <box size="${trunk_length} ${trunk_width} ${trunk_height}" />
+            </geometry>
+        </collision>
+        <inertial>
+            <origin rpy="0 0 0" xyz="${trunk_com_x} ${trunk_com_y} ${trunk_com_z}" />
+            <mass value="${trunk_mass}" />
+            <inertia ixx="${trunk_ixx}" ixy="${trunk_ixy}" ixz="${trunk_ixz}" iyy="${trunk_iyy}"
+                iyz="${trunk_iyz}" izz="${trunk_izz}" />
+        </inertial>
+    </link>
+    <joint name="imu_joint" type="fixed">
+        <parent link="trunk" />
+        <child link="imu_link" />
+        <origin rpy="0 0 0" xyz="0 0 0" />
+    </joint>
+    <link name="imu_link">
+        <inertial>
+            <mass value="0.001" />
+            <origin rpy="0 0 0" xyz="0 0 0" />
+            <inertia ixx="0.0001" ixy="0" ixz="0" iyy="0.0001" iyz="0" izz="0.0001" />
+        </inertial>
+        <visual>
+            <origin rpy="0 0 0" xyz="0 0 0" />
+            <geometry>
+                <box size="0.001 0.001 0.001" />
+            </geometry>
+        </visual>
+        <collision>
+            <origin rpy="0 0 0" xyz="0 0 0" />
+            <geometry>
+                <box size=".001 .001 .001" />
+            </geometry>
+        </collision>
+    </link>
+    <!-- Camera Link-->
+    <link name="camera_link">
+        <inertial>
+            <mass value="0.001" />
+            <origin rpy="0 0 0" xyz="0 0 0" />
+            <inertia ixx="0.0001" ixy="0" ixz="0" iyy="0.0001" iyz="0" izz="0.0001" />
+        </inertial>
+        <visual>
+            <origin rpy="0 0 0" xyz="0 0 0" />
+            <geometry>
+                <sphere radius="0.001" />
+            </geometry>
+            <material name="">
+                <color rgba="0.5 0 0 1" />
+            </material>
+        </visual>
+        <collision>
+            <origin rpy="0 0 0" xyz="0 0 0" />
+            <geometry>
+                <sphere radius="0.001" />
+            </geometry>
+        </collision>
+    </link>
+    <joint name="camera_joint" type="fixed">
+        <parent link="trunk" />
+        <child link="camera_link" />
+        <origin rpy="0 0 0" xyz="0.326 0 0.043" />
+    </joint>
+    <!-- <joint name="lidar_l1_joint" type="fixed">
+        <parent link="base_link"/>
+        <child link="lidar_l1_link"/>
+        <origin rpy="2.94 0 1.5705" xyz="0.25 -0.038 -0.03"/>
+    </joint>
+    <link name="lidar_l1_link">
+        <inertial>
+            <mass value="0.5"/>
+            <origin rpy="0 0 0" xyz="0 0 0"/>
+            <inertia ixx="0.01" ixy="0" ixz="0" iyy="0.01" iyz="0" izz="0.01"/>
+        </inertial>
+        <visual>
+            <origin rpy="0 0 0" xyz="0 0 0"/>
+            <geometry>
+                <mesh filename="file://$(find unitree_go2_description)/meshes/L1_4D_Lidar.dae" scale="1 1 1"/>
+            </geometry>
+            <material name="black">
+                <color rgba="0.0 0.0 0.0 1.0"/>
+            </material>
+        </visual>
+        <collision>
+            <origin rpy="0 0 0" xyz="0 0 0"/>
+            <geometry>
+                <mesh filename="file://$(find unitree_go2_description)/meshes/L1_4D_Lidar.dae" scale="1 1 1"/>
+            </geometry>
+            <material name="black">
+                <color rgba="0.0 0.0 0.0 1.0"/>
+            </material>
+        </collision>
+    </link> -->
+    <xacro:leg name="rf" mirror="-1" mirror_dae="False" front_hind="1" front_hind_dae="True" />
+    <xacro:leg name="lf" mirror="1" mirror_dae="True" front_hind="1" front_hind_dae="True" />
+    <xacro:leg name="rh" mirror="-1" mirror_dae="False" front_hind="-1" front_hind_dae="False" />
+    <xacro:leg name="lh" mirror="1" mirror_dae="True" front_hind="-1" front_hind_dae="False" />
+</robot>

File: install/unitree_go2_description/share/unitree_go2_description/urdf/velodyne.xacro (robot description, xacro)
@@ -1 +1,86 @@
-/home/ming/ros2_ws/src/unitree_go2/unitree_go2_description/urdf/velodyne.xacro
+<?xml version="1.0"?>
+<robot xmlns:xacro="http://www.ros.org/wiki/xacro">
+    <joint name="velodyne_base_mount_joint" type="fixed">
+        <origin rpy="0 0 0" xyz="0.2 0 0.08"/>
+        <parent link="base_link"/>
+        <child link="velodyne_base_link"/>
+    </joint>
+    <link name="velodyne_base_link">
+        <inertial>
+            <mass value="0.83"/>
+            <origin xyz="0 0 0.03585"/>
+            <inertia ixx="0.000908059425" ixy="0" ixz="0" iyy="0.000908059425" iyz="0" izz="0.0011049624"/>
+        </inertial>
+        <visual>
+            <geometry>
+                <mesh filename="file://$(find unitree_go2_description)/meshes/VLP16_base_1.dae"/>
+            </geometry>
+        </visual>
+        <visual>
+            <geometry>
+                <mesh filename="file://$(find unitree_go2_description)/meshes/VLP16_base_2.dae"/>
+            </geometry>
+        </visual>
+        <collision>
+            <origin rpy="0 0 0" xyz="0 0 0.03585"/>
+            <geometry>
+                <cylinder length="0.0717" radius="0.0516"/>
+            </geometry>
+        </collision>
+    </link>
+    <joint name="velodyne_base_scan_joint" type="fixed">
+        <origin rpy="0 0 0" xyz="0 0 0.0377"/>
+        <parent link="velodyne_base_link"/>
+        <child link="velodyne"/>
+    </joint>
+    <link name="velodyne">
+        <inertial>
+            <mass value="0.01"/>
+            <origin xyz="0 0 0"/>
+            <inertia ixx="1e-7" ixy="0" ixz="0" iyy="1e-7" iyz="0" izz="1e-7"/>
+        </inertial>
+        <visual>
+            <origin xyz="0 0 -0.0377"/>
+            <geometry>
+                <mesh filename="file://$(find unitree_go2_description)/meshes/VLP16_scan.dae"/>
+            </geometry>
+        </visual>
+    </link>
+    <!-- Gazebo Sim Velodyne Sensor plugin -->
+    <gazebo reference="velodyne">
+        <sensor name="velodyne-VLP16" type="gpu_lidar">
+            <topic>velodyne_points</topic>
+            <update_rate>10</update_rate>
+            <gz_frame_id>velodyne</gz_frame_id>
+            <lidar>
+                <scan>
+                    <horizontal>
+                        <samples>440</samples>
+                        <resolution>1</resolution>
+                        <min_angle>-3.14159</min_angle>
+                        <max_angle>3.14159</max_angle>
+                    </horizontal>
+                    <vertical>
+                        <samples>16</samples>
+                        <resolution>1</resolution>
+                        <min_angle>-0.261799</min_angle>
+                        <max_angle>0.261799</max_angle>
+                    </vertical>
+                </scan>
+                <range>
+                    <min>0.5</min>
+                    <max>131.0</max>
+                    <resolution>0.001</resolution>
+                </range>
+                <noise>
+                    <type>gaussian</type>
+                    <mean>0.0</mean>
+                    <stddev>0.008</stddev>
+                </noise>
+                <frame_id>velodyne</frame_id>
+            </lidar>
+            <visualize>true</visualize>
+            <always_on>1</always_on>
+        </sensor>
+    </gazebo>
+</robot>
